File: analog-mixer/hw/analog/analog_routed.kicad_pcb (KiCad board)
At the start: 4 copper layers, 129 x 137.5 mm, 400 parts, among them J1 SJ-43514-SMT, J10 GCT USB4085, J11 Модуль IP2326: VBUS, GND, BAT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, J2 SJ-43514-SMT, J3 SJ-43514-SMT, J4 SJ-43514-SMT, J5 SJ-43514-SMT, J6 SJ-43514-SMT MAIN, J7 SJ-43514-SMT SEND, J8 SJ-43514-SMT PHONES, J9 PBS-24 до цифрової плати, Q1 AO3401A, SW1 CTS 204-121ST, SW10 Cherry MX, SW11 Cherry MX, SW12 MSK12C02 вимикач живлення, SW2 Cherry MX, SW3 CTS 204-121ST, SW4 Cherry MX, SW5 CTS 204-121ST, SW6 Cherry MX, SW7 CTS 204-121ST, SW8 Cherry MX, SW9 CTS 204-121ST, U1 OPA1678, U10 DG413, U11 OPA1678, U12 DG413, U13 OPA1678, U14 OPA1678, U15 OPA1678, U16 OPA1678, U17 OPA1678, U18 OPA1678, U19 TL064AC, U2 DG413, U20 TL064AC, U21 TL064AC, U22 TL064AC, U23 TL064AC, U24 TL064AC, U25 MCP23017-E/SO, U26 USBLC6-2SC6, U27 CH340N, U28 LT1930ES5, U29 LT1931ES5, U3 OPA1678, U30 TPS62933O, U4 DG413, U5 OPA1678, U6 DG413, U7 OPA1678, U8 DG413, U9 OPA1678

Commit message: Адреса джерел на шовкографії обох плат (D9, CERN-OHL-S розд. 4)
- build_pcb.ATTRIB / add_attribution(), hw/pcb/add_silk.py для розведених плат
- panel.py: файл правил DRC — за іменем файлу (шлях analog-mixer/ ламав відбір)
- панель і hw/fab перезібрано; DRC: 0 розривів, нових зауважень немає

Co-Authored-By: Claude Opus 5.5 <noreply@anthropic.com>
Other:
- board text added: "based on github.com/stahlnow/mixerli"
- board text added: "github.com/heartpolik/hardware-pocket-mixer"
- board text added: "hardware-pocket-mixer Rev A CERN-OHL-S-2.0+"
Changed lines of the file:
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@@
 		(layer "Edge.Cuts")
+	)
+	(gr_text "hardware-pocket-mixer Rev A  CERN-OHL-S-2.0+"
+		(at 81.45 150.1 0)
+		(layer "B.SilkS")
+		(effects
+			(font
+				(size 1 1)
+				(thickness 0.15)
+			)
+			(justify mirror)
+		)
+	)
+	(gr_text "github.com/heartpolik/hardware-pocket-mixer"
+		(at 81.45 151.9 0)
+		(layer "B.SilkS")
+		(effects
+			(font
+				(size 1 1)
+				(thickness 0.15)
+			)
+			(justify mirror)
+		)
+	)
+	(gr_text "based on github.com/stahlnow/mixerli"
+		(at 81.45 153.7 0)
+		(layer "B.SilkS")
+		(effects
+			(font
+				(size 1 1)
+				(thickness 0.15)
+			)
+			(justify mirror)
+		)
 	)
 	(via
