File: analog-mixer/hw/digital/digital_routed.kicad_pcb (KiCad board)
At the start: 4 copper layers, 129 x 51.5 mm, 44 parts, among them J1 PLS-24 до аналогової плати, SW1 EC12D (30/15) з кнопкою, U1 ESP32-C3 SuperMini, U2 ADS7828, U3 SN74AHCT1G125DBV

Commit message: Адреса джерел на шовкографії обох плат (D9, CERN-OHL-S розд. 4)
- build_pcb.ATTRIB / add_attribution(), hw/pcb/add_silk.py для розведених плат
- panel.py: файл правил DRC — за іменем файлу (шлях analog-mixer/ ламав відбір)
- панель і hw/fab перезібрано; DRC: 0 розривів, нових зауважень немає

Co-Authored-By: Claude Opus 5.5 <noreply@anthropic.com>
Other:
- board text added: "based on github.com/stahlnow/mixerli"
- board text added: "github.com/heartpolik/hardware-pocket-mixer"
- board text added: "hardware-pocket-mixer Rev A CERN-OHL-S-2.0+"
Changed lines of the file:
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@@
 		(layer "Edge.Cuts")
+	)
+	(gr_text "hardware-pocket-mixer Rev A  CERN-OHL-S-2.0+"
+		(at 52.7 31.35 0)
+		(layer "F.SilkS")
+		(effects
+			(font
+				(size 1 1)
+				(thickness 0.15)
+			)
+		)
+	)
+	(gr_text "github.com/heartpolik/hardware-pocket-mixer"
+		(at 52.7 33.15 0)
+		(layer "F.SilkS")
+		(effects
+			(font
+				(size 1 1)
+				(thickness 0.15)
+			)
+		)
+	)
+	(gr_text "based on github.com/stahlnow/mixerli"
+		(at 52.7 34.95 0)
+		(layer "F.SilkS")
+		(effects
+			(font
+				(size 1 1)
+				(thickness 0.15)
+			)
+		)
 	)
 	(segment
