File: digital-mixer/hw/main/main.kicad_sch (KiCad schematic)
At the start: 186 parts, among them J1 GCT USB4085, J2 LiPo 1S 3000 mAh (з платою за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, J3 IN1 SJ-43514-SMT, J4 IN2 SJ-43514-SMT, J5 IN3 SJ-43514-SMT, J6 IN4 SJ-43514-SMT, J7 MAIN OUT SJ-43514-SMT, J8 AUX OUT SJ-43514-SMT, J9 PHONES SJ-43514-SMT, Q1 AO3401A, SW1 MSK12C02 вимикач, SW10 EC11 ch3.1, SW11 EC11 ch3.2, SW12 EC11 ch3.3, SW13 Mute 3 Kailh PG1350, SW14 EC11 ch4.1, SW15 EC11 ch4.2, SW16 EC11 ch4.3, SW17 Mute 4 Kailh PG1350, SW18 EC11 master, SW19 FX1 Kailh PG1350, SW2 EC11 ch1.1, SW20 FX2 Kailh PG1350, SW21 AUX Kailh PG1350, SW22 CUE Kailh PG1350, SW23 SHIFT Kailh PG1350, SW3 EC11 ch1.2, SW4 EC11 ch1.3, SW5 Mute 1 Kailh PG1350, SW6 EC11 ch2.1, SW7 EC11 ch2.2, SW8 EC11 ch2.3, SW9 Mute 2 Kailh PG1350, U1 Teensy 4.1, U10 PCM5102A, U11 TPA6132A2, U12 MCP23017-E/SO, U13 MCP23017-E/SO, U2 USBLC6-2SC6, U3 TP4056, U4 TPS63802, U5 LP5907MFX-3.3, U6 PCM1865, U7 PCM1865, U8 PCM5102A, U9 PCM5102A

Commit message: digital-mixer: дисплей GMT147SPI, кнопки TSF-1266, живлення кнопкою з фіксацією (DM16-DM18)
- без адресних LED; FX I/FX II/AUX/CUE на вільних виводах MCP23017, SPI дисплея на Teensy
- кнопка живлення 7x7 DPDT на EN TPS63802; ERC 0 помилок, нетлист без одиночних кіл
- макет 108 x 97 мм; живлення 1,48 W -> 6,8 год на 3000 mAh

Co-Authored-By: Claude Opus 5.5 <noreply@anthropic.com>
Parts:
- removed C82, C83, C84: 100n, Capacitor_SMD:C_0805_2012Metric, symbol Device:C
- removed C85: 10u, Capacitor_SMD:C_1206_3216Metric, symbol Device:C
- removed DS1: OLED 0.96 128x64 I2C, pocket-digital:OLED_0.96in_128x64_I2C_4pin, symbol Connector_Generic:Conn_01x04
- removed LED1: SK6812MINI-E mute1, LED_SMD:LED_SK6812MINI-E_3.2x2.8mm_P1.5mm_ReverseMount, symbol LED:SK6812MINI-E
- removed LED2: SK6812MINI-E mute2, LED_SMD:LED_SK6812MINI-E_3.2x2.8mm_P1.5mm_ReverseMount, symbol LED:SK6812MINI-E
- removed LED3: SK6812MINI-E mute3, LED_SMD:LED_SK6812MINI-E_3.2x2.8mm_P1.5mm_ReverseMount, symbol LED:SK6812MINI-E
- removed LED4: SK6812MINI-E mute4, LED_SMD:LED_SK6812MINI-E_3.2x2.8mm_P1.5mm_ReverseMount, symbol LED:SK6812MINI-E
- removed R42: 33, Resistor_SMD:R_0805_2012Metric, symbol Device:R
- removed SW1: MSK12C02 вимикач, pocket-digital:SW_Slide_SPDT_SHOUHAN_MSK12C02_RightAngle, symbol Switch:SW_SPDT
- added DS1: GMT147SPI 1.47in 172x320, pocket-digital:LCD_GMT147SPI, symbol Connector_Generic:Conn_01x08
- added SW1: Power 7x7 DPDT self-lock, pocket-digital:SW_Push_Latching_DPDT_7x7mm, symbol Switch:SW_DPDT_x2
- C81: value 100n -> 10u; footprint Capacitor_SMD:C_0805_2012Metric -> Capacitor_SMD:C_1206_3216Metric; Decouples LED1 -> (none)
- SW13: value Mute 3 Kailh PG1350 -> Mute 3 TSF-1266; footprint pocket-digital:Kailh_Choc_PG1350 -> pocket-digital:SW_TSF-1266_6x6mm_SMD
- SW17: value Mute 4 Kailh PG1350 -> Mute 4 TSF-1266; footprint pocket-digital:Kailh_Choc_PG1350 -> pocket-digital:SW_TSF-1266_6x6mm_SMD
- SW19: value FX1 Kailh PG1350 -> FX1 TSF-1266; footprint pocket-digital:Kailh_Choc_PG1350 -> pocket-digital:SW_TSF-1266_6x6mm_SMD
- SW20: value FX2 Kailh PG1350 -> FX2 TSF-1266; footprint pocket-digital:Kailh_Choc_PG1350 -> pocket-digital:SW_TSF-1266_6x6mm_SMD
- SW21: value AUX Kailh PG1350 -> AUX TSF-1266; footprint pocket-digital:Kailh_Choc_PG1350 -> pocket-digital:SW_TSF-1266_6x6mm_SMD
- SW22: value CUE Kailh PG1350 -> CUE TSF-1266; footprint pocket-digital:Kailh_Choc_PG1350 -> pocket-digital:SW_TSF-1266_6x6mm_SMD
- SW23: value SHIFT Kailh PG1350 -> SHIFT TSF-1266; footprint pocket-digital:Kailh_Choc_PG1350 -> pocket-digital:SW_TSF-1266_6x6mm_SMD
- SW5: value Mute 1 Kailh PG1350 -> Mute 1 TSF-1266; footprint pocket-digital:Kailh_Choc_PG1350 -> pocket-digital:SW_TSF-1266_6x6mm_SMD
- SW9: value Mute 2 Kailh PG1350 -> Mute 2 TSF-1266; footprint pocket-digital:Kailh_Choc_PG1350 -> pocket-digital:SW_TSF-1266_6x6mm_SMD
Connections:
- net +3V3: now also C81.1, DS1.1 (Pin_1)
- net +4V2: no longer C81.1
- net BTN_AUX: now also U13.28 (GPA7); no longer U1.14 (12_MISO_MQSL)
- net BTN_CUE: now also U13.8 (GPB7); no longer U1.20 (28_RX7)
- net BTN_FX1: now also U12.28 (GPA7); no longer U1.12 (10_CS_MQSR)
- net BTN_FX2: now also U12.8 (GPB7); no longer U1.13 (11_MOSI_CTX1)
- net GND: now also DS1.2 (Pin_2), SW1.3 (C)
- net PWR_EN: now also SW1.2 (B)
- net VSYS: now also SW1.1 (A)
- net LCD_DC: now reaches U1.32 (40_A16)
- net LCD_DC: now also DS1.7 (Pin_7)
- net LCD_RES: now reaches U1.33 (41_A17)
- net LCD_RES: now also DS1.6 (Pin_6)
- net LCD_SCK: now reaches U1.35 (13_SCK_LED)
- net LCD_SCK: now also DS1.3 (Pin_3)
- net LED_DATA_3V3: no longer names the net of U1.27 (35_TX8)
- new net LCD_BLK: DS1.8 (Pin_8), U1.20 (28_RX7)
- new net LCD_CS: DS1.5 (Pin_5), U1.12 (10_CS_MQSR)
- new net LCD_MOSI: DS1.4 (Pin_4), U1.13 (11_MOSI_CTX1)
- no-connect marks 60 -> 57
Other:
- note added: "Buck-boost TPS63802 → +4V2 (DM11). R1/R2 = 665k/91k → 4,15 V (VFB 0,5 V, табл. 10-5); L 0,47 µH XFL4015; C 10 µF вх., 2×22 µF вих. (>3,6 V). Вимикач — кнопка з фіксацією 7×7 на EN (DM17)"
- note added: "MCP23017 #1 (I²C2, 0x20): енкодери каналів 1, 2 (A/B), Mute, кнопки FX/AUX/CUE (GPx7); внутрішні підтяжки 100k, INTA/INTB дзеркальні → один INT"
- note added: "MCP23017 #2 (I²C2, 0x21): енкодери каналів 3, 4 (A/B), Mute, кнопки FX/AUX/CUE (GPx7); внутрішні підтяжки 100k, INTA/INTB дзеркальні → один INT"
- note added: "Канал 1: 3 енкодери EC11 (шари EQ / посили / канал, DM6), фейдер 35 мм (DM8), Mute — тактова кнопка TSF-1266 (DM16)"
- note added: "Канал 2: 3 енкодери EC11 (шари EQ / посили / канал, DM6), фейдер 35 мм (DM8), Mute — тактова кнопка TSF-1266 (DM16)"
- note added: "Канал 3: 3 енкодери EC11 (шари EQ / посили / канал, DM6), фейдер 35 мм (DM8), Mute — тактова кнопка TSF-1266 (DM16)"
- note added: "Канал 4: 3 енкодери EC11 (шари EQ / посили / канал, DM6), фейдер 35 мм (DM8), Mute — тактова кнопка TSF-1266 (DM16)"
- note added: "Майстер: енкодер EC11 з кнопкою, кнопки FX I, FX II, AUX, CUE, SHIFT (TSF-1266); дисплей GMT147SPI 1,47" 172×320 ST7789, SPI (DM18) — порядок виводів модуля ПЕРЕВІРИТИ"
- note removed: "Buck-boost TPS63802 → +4V2 (DM11). R1/R2 = 665k/91k → 4,15 V (VFB 0,5 V, табл. 10-5); L 0,47 µH XFL4015; C 10 µF вх., 2×22 µF вих. (>3,6 V). Вимикач MSK12C02 — на EN"
- note removed: "LED під Mute: 4 × SK6812MINI-E (зворотний монтаж під вікном Choc), живлення +4V2 (≥ 3,7 V); DIN 3,3 V ≥ 0,7·VDD = 2,9 V — запас `ПЕРЕВІРИТИ`"
- note removed: "MCP23017 #1 (I²C2, 0x20): енкодери каналів 1, 2 (A/B) і Mute; внутрішні підтяжки 100k, INTA/INTB дзеркальні → один INT"
- note removed: "MCP23017 #2 (I²C2, 0x21): енкодери каналів 3, 4 (A/B) і Mute; внутрішні підтяжки 100k, INTA/INTB дзеркальні → один INT"
- note removed: "Канал 1: 3 енкодери EC11 (шари EQ / посили / канал, DM6), фейдер 35 мм (DM8), Mute — Kailh Choc PG1350 з SK6812MINI-E під ним"
- note removed: "Канал 2: 3 енкодери EC11 (шари EQ / посили / канал, DM6), фейдер 35 мм (DM8), Mute — Kailh Choc PG1350 з SK6812MINI-E під ним"
- note removed: "Канал 3: 3 енкодери EC11 (шари EQ / посили / канал, DM6), фейдер 35 мм (DM8), Mute — Kailh Choc PG1350 з SK6812MINI-E під ним"
- note removed: "Канал 4: 3 енкодери EC11 (шари EQ / посили / канал, DM6), фейдер 35 мм (DM8), Mute — Kailh Choc PG1350 з SK6812MINI-E під ним"
- note removed: "Майстер: енкодер EC11 з кнопкою, кнопки FX I, FX II, AUX, CUE, SHIFT (Choc, внутр. підтяжка Teensy), OLED"

Commit message: digital-mixer: MIDI OUT TRS Type A (DM20)
Co-Authored-By: Claude Opus 5.5 <noreply@anthropic.com>
Parts:
- added J10: MIDI OUT SJ-43514-SMT, pocket-digital:CUI_SJ-43514-SMT_TRRS_Horizontal, symbol pocket-digital:AudioJack_TRRS_SJ-43514
- added R42: 33 0.5W, Resistor_SMD:R_2010_5025Metric, symbol Device:R
- added R43: 10 0.25W, Resistor_SMD:R_1206_3216Metric, symbol Device:R
Connections:
- net +3V3: now also R42.1
- net GND: now also J10.1 (S), J10.4 (R2)
- net MIDI_TX: now reaches U1.27 (35_TX8)
- net MIDI_TX: now also R43.1
- new net MIDI_SINK: J10.2 (T), R43.2
- new net MIDI_SRC: J10.3 (R1), R42.2
- no-connect marks 57 -> 56
Other:
- note added: "MIDI OUT, TRS Type A (DM20): кінчик = DIN 5 (через RC 10 Ω від UART), кільце = DIN 4 (RA 33 Ω від +3,3 V), гільза = DIN 2 / GND. Значення для 3,3 V — MIDI 1.0 Electrical Spec Update, рис. 1"

Commit message: digital-mixer: footprint (Teensy 4.1, TPS63802, XFL4015, заглушки), розстановка WIP, DM21-DM23
- hw/lib/gen_footprints.py: Teensy41_SMD (PJRC), VSON-HR-10 (TI DLA0010A), XFL4015 (Coilcraft),
  M2; заглушки TSF-1266, кнопки 7x7, GMT147SPI - до креслень / вимірів
- GMT147SPI: порядок виводів за кресленням продавця
- hw/pcb/pcbkit.py (з Rev A), build_pcb.py: перша розстановка, отвори M2 у кутах;
  конфлікт THT-виводів керування з джеками й Teensy знизу - компоновку треба змінити

Co-Authored-By: Claude Opus 5.5 <noreply@anthropic.com>
Connections:
- net +3V3: now also DS1.2 (Pin_2); no longer DS1.1 (Pin_1)
- net GND: now also DS1.1 (Pin_1); no longer DS1.2 (Pin_2)
- net LCD_CS: now also DS1.7 (Pin_7); no longer DS1.5 (Pin_5)
- net LCD_DC: now also DS1.6 (Pin_6); no longer DS1.7 (Pin_7)
- net LCD_RES: now also DS1.5 (Pin_5); no longer DS1.6 (Pin_6)
Other:
- note added: "Майстер: енкодер EC11 з кнопкою, кнопки FX I, FX II, AUX, CUE, SHIFT (TSF-1266); дисплей GMT147SPI 1,47" 172×320 ST7789P3, SPI, на гребінці (DM18, DM23); виводи — за кресленням продавця"
- note removed: "Майстер: енкодер EC11 з кнопкою, кнопки FX I, FX II, AUX, CUE, SHIFT (TSF-1266); дисплей GMT147SPI 1,47" 172×320 ST7789, SPI (DM18) — порядок виводів модуля ПЕРЕВІРИТИ"

Commit message: digital-mixer: двошарова плата розведена (DRC: 0 розривів, 0 порушень по міді)
- Teensy праворуч спереду (microSD у правий торець), USB-C і PHONES на фронті: USB D+/D- ~30 мм
- блок TPS63802 за прикладом TI, доріжки зафіксовані; конденсатори біля виводів
- footprint TSF-1266 без подвійного courtyard; route_pcb зберігає зафіксовані доріжки
- docs/04-pcb.md

Co-Authored-By: Claude Opus 5.5 <noreply@anthropic.com>
Parts:
- U11: footprint Package_DFN_QFN:WQFN-16-1EP_3x3mm_P0.5mm_EP1.6x1.6mm_ThermalVias -> Package_DFN_QFN:WQFN-16-1EP_3x3mm_P0.5mm_EP1.6x1.6mm
- U3: footprint Package_SO:SOIC-8-1EP_3.9x4.9mm_P1.27mm_EP2.41x3.3mm_ThermalVias -> Package_SO:SOIC-8-1EP_3.9x4.9mm_P1.27mm_EP2.41x3.3mm

Commit message: digital-mixer: компоновка C (DM25-DM30), SMD-енкодери, USB4110, розводка 0 помилок
- компоновка C: колонки каналів на одних осях, ON / дисплей / MASTER в один ряд,
  Teensy у передньому правому куті, виходи на правому торці, M2 у чотирьох кутах
- EC12SY SMD з кнопками (DM26) + третій MCP23017; кнопку CUE прибрано (DM28)
- кнопка живлення 5,8 мм SMD (DM27), USB-C GCT USB4110 SMD (DM30), JST PH SMD
- 33 Ω на тактах I2S / TDM (DM29); такти 60-73 мм замість ~110
- 3D-моделі для всіх власних і стокових footprint без моделі (hw/lib/gen_3d.py)
- common: route_pcb --hole-keep, rip_near.py, параметри проєкту в kisch
- DRC: 0 порушень, 0 нез'єднаних, 0 розбіжностей зі схемою; ERC 0

Co-Authored-By: Claude Opus 5.5 <noreply@anthropic.com>
Parts:
- removed J2: LiPo 1S 3000 mAh (з платою захисту), Connector_JST:JST_PH_B2B-PH-K_1x02_P2.00mm_Vertical, symbol Connector_Generic:Conn_01x02
- removed SW10: EC11 ch3.1, Rotary_Encoder:RotaryEncoder_Alps_EC11E_Vertical_H20mm, symbol Device:RotaryEncoder
- removed SW11: EC11 ch3.2, Rotary_Encoder:RotaryEncoder_Alps_EC11E_Vertical_H20mm, symbol Device:RotaryEncoder
- removed SW12: EC11 ch3.3, Rotary_Encoder:RotaryEncoder_Alps_EC11E_Vertical_H20mm, symbol Device:RotaryEncoder
- removed SW14: EC11 ch4.1, Rotary_Encoder:RotaryEncoder_Alps_EC11E_Vertical_H20mm, symbol Device:RotaryEncoder
- removed SW15: EC11 ch4.2, Rotary_Encoder:RotaryEncoder_Alps_EC11E_Vertical_H20mm, symbol Device:RotaryEncoder
- removed SW16: EC11 ch4.3, Rotary_Encoder:RotaryEncoder_Alps_EC11E_Vertical_H20mm, symbol Device:RotaryEncoder
- removed SW18: EC11 master, Rotary_Encoder:RotaryEncoder_Alps_EC11E-Switch_Vertical_H20mm, symbol Device:RotaryEncoder_Switch
- removed SW2: EC11 ch1.1, Rotary_Encoder:RotaryEncoder_Alps_EC11E_Vertical_H20mm, symbol Device:RotaryEncoder
- removed SW23: SHIFT TSF-1266, pocket-digital:SW_TSF-1266_6x6mm_SMD, symbol Switch:SW_Push
- removed SW3: EC11 ch1.2, Rotary_Encoder:RotaryEncoder_Alps_EC11E_Vertical_H20mm, symbol Device:RotaryEncoder
- removed SW4: EC11 ch1.3, Rotary_Encoder:RotaryEncoder_Alps_EC11E_Vertical_H20mm, symbol Device:RotaryEncoder
- removed SW6: EC11 ch2.1, Rotary_Encoder:RotaryEncoder_Alps_EC11E_Vertical_H20mm, symbol Device:RotaryEncoder
- removed SW7: EC11 ch2.2, Rotary_Encoder:RotaryEncoder_Alps_EC11E_Vertical_H20mm, symbol Device:RotaryEncoder
- removed SW8: EC11 ch2.3, Rotary_Encoder:RotaryEncoder_Alps_EC11E_Vertical_H20mm, symbol Device:RotaryEncoder
- added C82: 10u, Capacitor_SMD:C_1206_3216Metric, symbol Device:C
- added J2: LiPo 1S 3000 mAh (з платою захисту), Connector_JST:JST_PH_S2B-PH-SM4-TB_1x02-1MP_P2.00mm_Horizontal, symbol Connector_Generic_MountingPin:Conn_01x02_MountingPin
- added R44, R45, R46: 470, Resistor_SMD:R_0805_2012Metric, symbol Device:R
- added R47: 33 0.5W, Resistor_SMD:R_2010_5025Metric, symbol Device:R
- added R48: 10 0.25W, Resistor_SMD:R_1206_3216Metric, symbol Device:R
- added SW10: EC12SY ch3.1, pocket-digital:RotaryEncoder_EC12SY_SMD, symbol Device:RotaryEncoder_Switch_MP
- added SW11: EC12SY ch3.2, pocket-digital:RotaryEncoder_EC12SY_SMD, symbol Device:RotaryEncoder_Switch_MP
- added SW12: EC12SY ch3.3, pocket-digital:RotaryEncoder_EC12SY_SMD, symbol Device:RotaryEncoder_Switch_MP
- added SW14: EC12SY ch4.1, pocket-digital:RotaryEncoder_EC12SY_SMD, symbol Device:RotaryEncoder_Switch_MP
- added SW15: EC12SY ch4.2, pocket-digital:RotaryEncoder_EC12SY_SMD, symbol Device:RotaryEncoder_Switch_MP
- added SW16: EC12SY ch4.3, pocket-digital:RotaryEncoder_EC12SY_SMD, symbol Device:RotaryEncoder_Switch_MP
- added SW18: EC12SY master, pocket-digital:RotaryEncoder_EC12SY_SMD, symbol Device:RotaryEncoder_Switch_MP
- added SW2: EC12SY ch1.1, pocket-digital:RotaryEncoder_EC12SY_SMD, symbol Device:RotaryEncoder_Switch_MP
- added SW3: EC12SY ch1.2, pocket-digital:RotaryEncoder_EC12SY_SMD, symbol Device:RotaryEncoder_Switch_MP
- added SW4: EC12SY ch1.3, pocket-digital:RotaryEncoder_EC12SY_SMD, symbol Device:RotaryEncoder_Switch_MP
- added SW6: EC12SY ch2.1, pocket-digital:RotaryEncoder_EC12SY_SMD, symbol Device:RotaryEncoder_Switch_MP
- added SW7: EC12SY ch2.2, pocket-digital:RotaryEncoder_EC12SY_SMD, symbol Device:RotaryEncoder_Switch_MP
- added SW8: EC12SY ch2.3, pocket-digital:RotaryEncoder_EC12SY_SMD, symbol Device:RotaryEncoder_Switch_MP
- added U14: MCP23017-E/SO, Package_SO:SOIC-28W_7.5x17.9mm_P1.27mm, symbol Interface_Expansion:MCP23017x-x-SO
- C71, C72, C73, C74: Decouples (none) -> U11
- C77: Decouples (none) -> U14
- C81: value 10u -> 100n; footprint Capacitor_SMD:C_1206_3216Metric -> Capacitor_SMD:C_0805_2012Metric
- J1: value GCT USB4085 -> GCT USB4110-GF-A; footprint Connector_USB:USB_C_Receptacle_GCT_USB4085 -> Connector_USB:USB_C_Receptacle_GCT_USB4110
- R10: value 5.1k -> 10k
- R11: value 2.4k -> 10k
- R12, R13: value 1k -> 100k
- R14: value 100k -> 5.1k
- R15: value 665k -> 5.1k
- R16: value 91k -> 2.4k
- R17, R18: value 100k -> 1k
- R19, R23, R25, R32, R34: value 10k -> 100k
- R20: value 100k -> 665k
- R21: value 10k -> 91k
- R24, R33: value 100k -> 10k
- R26, R35: value 33 -> 10k
- R31, R7, R8: value 100k -> 33
- R36, R38: value 470 -> 100k
- R37, R39: value 470 -> 10k
- R40: value 470 -> 33
- R42: value 33 0.5W -> 470; footprint Resistor_SMD:R_2010_5025Metric -> Resistor_SMD:R_0805_2012Metric
- R43: value 10 0.25W -> 470; footprint Resistor_SMD:R_1206_3216Metric -> Resistor_SMD:R_0805_2012Metric
- R5, R6: value 10k -> 33
- R9: value 5.1k -> 33
- SW1: value Power 7x7 DPDT self-lock -> Power 5.8mm DPDT self-lock SMD; footprint pocket-digital:SW_Push_Latching_DPDT_7x7mm -> pocket-digital:SW_Push_Latching_DPDT_5.8mm_SMD
- SW22: value CUE TSF-1266 -> SHIFT TSF-1266
Connections:
- net +3V3: now also C77.1, C82.1, R47.1, U14.16 (A1), U14.18 (~{RESET}), U14.9 (V_{DD}); no longer C81.1, R42.1
- net +4V2: now also R20.1; no longer R15.1
- net ADC1_DOUT: now also R31.1; no longer R26.1
- net ADC2_DOUT: now also R40.1; no longer R35.1
- net ADC_BCK: now also R7.2; no longer U1.6 (4_BCLK2)
- net ADC_DOUT: now also R31.2, R40.2; no longer R26.2, R35.2
- net ADC_LRCK: now also R8.2; no longer U1.5 (3_LRCLK2)
- net ADC_MCLK: now also R9.2; no longer U1.25 (33_MCLK2)
- net AUX_L: now also R43.2; no longer R38.2
- net AUX_OL: now also R43.1; no longer R38.1
- net AUX_OR: now also R44.1; no longer R39.1
- net AUX_R: now also R44.2; no longer R39.2
- net BAT+: now also J2.1 (Pin_1)
- net BB_FB: now also R20.2, R21.1; no longer R15.2, R16.1
- net BTN_AUX: now also U14.27 (GPA6); no longer U13.28 (GPA7)
- net BTN_FX1: now also U14.28 (GPA7); no longer U12.28 (GPA7)
- net BTN_FX2: now also U14.7 (GPB6); no longer U12.8 (GPB7)
- net BTN_SHIFT: now also SW22.1
- net CC1: now also R14.1; no longer R9.1
- net CC2: now also R15.1; no longer R10.1
- net CHG_LED_GA: now also R18.2; no longer R13.2
- net CHG_LED_RA: now also R17.2; no longer R12.2
- net CHG_PROG: now also R16.1; no longer R11.1
- net CUE_L: now also R45.2; no longer R40.2
- net CUE_OL: now also R45.1; no longer R40.1
- net CUE_OR: now also R46.1; no longer R41.1
- net CUE_R: now also R46.2; no longer R41.2
- net DAC_BCK: now also R5.2; no longer U1.43 (21_A7_RX5_BCLK1)
- net DAC_LRCK: now also R6.2; no longer U1.42 (20_A6_TX5_LRCLK1)
- net DAC_XSMT: now also R10.1; no longer R5.1
- net ENC1_1_A: now also SW2.A
- net ENC1_1_B: now also SW2.B
- net ENC1_2_A: now also SW3.A
- net ENC1_2_B: now also SW3.B
- net ENC1_3_A: now also SW4.A
- net ENC1_3_B: now also SW4.B
- net ENC2_1_A: now also SW6.A
- net ENC2_1_B: now also SW6.B
- net ENC2_2_A: now also SW7.A
- net ENC2_2_B: now also SW7.B
- net ENC2_3_A: now also SW8.A
- net ENC2_3_B: now also SW8.B
- net ENC3_1_A: now also SW10.A
- net ENC3_1_B: now also SW10.B
- net ENC3_2_A: now also SW11.A
- net ENC3_2_B: now also SW11.B
- net ENC3_3_A: now also SW12.A
- net ENC3_3_B: now also SW12.B
- net ENC4_1_A: now also SW14.A
- net ENC4_1_B: now also SW14.B
- net ENC4_2_A: now also SW15.A
- net ENC4_2_B: now also SW15.B
- net ENC4_3_A: now also SW16.A
- net ENC4_3_B: now also SW16.B
- net ENC_M_A: now also SW18.A
- net ENC_M_B: now also SW18.B
- net ENC_M_SW: now also SW18.S1
- net FADER1: now also C78.1; no longer C77.1
- net FADER2: now also C79.1; no longer C78.1
- net FADER3: now also C80.1; no longer C79.1
- net FADER4: now also C81.1; no longer C80.1
- net GND: now also R13.2, R15.2, R19.2, R21.2, R23.2, R25.2, R32.2, R34.2, R36.2, R38.2, SW1.1 (A), C82.2, J2.2 (Pin_2), J2.MP (MountPin), SW10.C, SW10.MP, SW10.S2, SW11.C, SW11.MP, SW11.S2, SW12.C, SW12.MP, SW12.S2, SW14.C, SW14.MP, SW14.S2, SW15.C, SW15.MP, SW15.S2, SW16.C, SW16.MP, SW16.S2, SW18.C, SW18.MP, SW18.S2, SW2.C, SW2.MP, SW2.S2, SW3.C, SW3.MP, SW3.S2, SW4.C, SW4.MP, SW4.S2, SW6.C, SW6.MP, SW6.S2, SW7.C, SW7.MP, SW7.S2, SW8.C, SW8.MP, SW8.S2, U14.10 (V_{SS}), U14.15 (A0), U14.17 (A2); no longer R17.2, R18.2, R20.2, R24.2, R31.2, R33.2, R5.2, R6.2, R8.2, R9.2, SW1.3 (C)
- net HP_EN: now also R11.1; no longer R6.1
- net I2C2_SCL: now also U14.12 (SCK)
- net I2C2_SDA: now also U14.13 (SDA)
- net IN1_LS: now also R24.2; no longer R19.2
- net IN1_R: now also R25.1, R26.1; no longer R20.1, R21.1
- net IN1_RS: now also R26.2; no longer R21.2
- net IN1_T: now also R23.1, R24.1; no longer R18.1, R19.1
- net IN2_LS: now also R28.2; no longer R23.2
- net IN2_R: now also R29.1, R30.1; no longer R24.1, R25.1
- net IN2_RS: now also R30.2; no longer R25.2
- net IN2_T: now also R27.1, R28.1; no longer R22.1, R23.1
- net IN3_LS: now also R33.2; no longer R28.2
- net IN3_R: now also R34.1, R35.1; no longer R29.1, R30.1
- net IN3_RS: now also R35.2; no longer R30.2
- net IN3_T: now also R32.1, R33.1; no longer R27.1, R28.1
- net IN4_LS: now also R37.2; no longer R32.2
- net IN4_R: now also R38.1, R39.1; no longer R33.1, R34.1
- net IN4_RS: now also R39.2; no longer R34.2
- net IN4_T: now also R36.1, R37.1; no longer R31.1, R32.1
- net MAIN_L: now also R41.2; no longer R36.2
- net MAIN_OL: now also R41.1; no longer R36.1
- net MAIN_OR: now also R42.1; no longer R37.1
- net MAIN_R: now also R42.2; no longer R37.2
- net MIDI_SINK: now also R48.2; no longer R43.2
- net MIDI_SRC: now also R47.2; no longer R42.2
- net MIDI_TX: now also R48.1; no longer R43.1
- net PWR_EN: now also R22.1; no longer R17.1
- net VBAT_SENSE: now also R12.2, R13.1; no longer R7.2, R8.1
- net VBUS: now also R17.1, R18.1, R19.1; no longer R12.1, R13.1, R14.1
- net VSYS: now also R12.1, SW1.3 (C); no longer R7.1, SW1.1 (A)
- net MCP3_INT: now reaches U1.44 (22_A8_CTX1)
- net MCP3_INT: now also U14.20 (INTA)
- net BTN_CUE: no longer names the net of U13.8 (GPB7)
- net BTN_CUE: no longer SW22.1
- new net ADC_BCK_T: R7.1, U1.6 (4_BCLK2)
- new net ADC_LRCK_T: R8.1, U1.5 (3_LRCLK2)
- new net ADC_MCLK_T: R9.1, U1.25 (33_MCLK2)
- new net DAC_BCK_T: R5.1, U1.43 (21_A7_RX5_BCLK1)
- new net DAC_LRCK_T: R6.1, U1.42 (20_A6_TX5_LRCLK1)
- new net ENC1_1_SW: SW2.S1, U14.21 (GPA0)
- new net ENC1_2_SW: SW3.S1, U14.22 (GPA1)
- new net ENC1_3_SW: SW4.S1, U14.23 (GPA2)
- new net ENC2_1_SW: SW6.S1, U14.24 (GPA3)
- new net ENC2_2_SW: SW7.S1, U14.25 (GPA4)
- new net ENC2_3_SW: SW8.S1, U14.26 (GPA5)
- new net ENC3_1_SW: SW10.S1, U14.1 (GPB0)
- new net ENC3_2_SW: SW11.S1, U14.2 (GPB1)
- new net ENC3_3_SW: SW12.S1, U14.3 (GPB2)
- new net ENC4_1_SW: SW14.S1, U14.4 (GPB3)
- new net ENC4_2_SW: SW15.S1, U14.5 (GPB4)
- new net ENC4_3_SW: SW16.S1, U14.6 (GPB5)
- no-connect marks 56 -> 63
Other:
- note added: "Buck-boost TPS63802 → +4V2 (DM11). R1/R2 = 665k/91k → 4,15 V (VFB 0,5 V, табл. 10-5); L 0,47 µH XFL4015; C 10 µF вх., 2×22 µF вих. (>3,6 V). Вимикач — кнопка з фіксацією 5,8 мм на EN (DM27)"
- note added: "MCP23017 #1 (I²C2, 0x20): енкодери каналів 1, 2 (A/B), Mute; GPx7 вільні; внутрішні підтяжки 100k, INTA/INTB дзеркальні → один INT"
- note added: "MCP23017 #2 (I²C2, 0x21): енкодери каналів 3, 4 (A/B), Mute; GPx7 вільні; внутрішні підтяжки 100k, INTA/INTB дзеркальні → один INT"
- note added: "MCP23017 #3 (I²C2, 0x22): кнопки 12 енкодерів каналів (DM28: натискання — фільтр / компресор, скидання значення) і кнопки AUX, FX I, FX II (GPA6, GPA7, GPB6) — найближчий до правої колонки; GPB7 вільний"
- note added: "USB-C (GCT USB4110-GF-A, повністю SMD — під MASTER, DM25): аудіо, MIDI, заряд. CC 5,1k — пристрій-споживач; ESD USBLC6"
- note added: "Канал 1: 3 енкодери EC12SY SMD з кнопкою (шари EQ / посили / канал, DM6, DM26), фейдер 35 мм (DM8), Mute — тактова кнопка TSF-1266 (DM16)"
- note added: "Канал 2: 3 енкодери EC12SY SMD з кнопкою (шари EQ / посили / канал, DM6, DM26), фейдер 35 мм (DM8), Mute — тактова кнопка TSF-1266 (DM16)"
- note added: "Канал 3: 3 енкодери EC12SY SMD з кнопкою (шари EQ / посили / канал, DM6, DM26), фейдер 35 мм (DM8), Mute — тактова кнопка TSF-1266 (DM16)"
- note added: "Канал 4: 3 енкодери EC12SY SMD з кнопкою (шари EQ / посили / канал, DM6, DM26), фейдер 35 мм (DM8), Mute — тактова кнопка TSF-1266 (DM16)"
- note added: "Майстер: енкодер EC12SY з кнопкою, кнопки AUX, FX I, FX II, SHIFT (TSF-1266; CUE = SHIFT + Mute, DM28); дисплей GMT147SPI 1,47" 172×320 ST7789P3, SPI, на гребінці (DM18, DM23); виводи — за кресленням продавця"
- note removed: "Buck-boost TPS63802 → +4V2 (DM11). R1/R2 = 665k/91k → 4,15 V (VFB 0,5 V, табл. 10-5); L 0,47 µH XFL4015; C 10 µF вх., 2×22 µF вих. (>3,6 V). Вимикач — кнопка з фіксацією 7×7 на EN (DM17)"
- note removed: "MCP23017 #1 (I²C2, 0x20): енкодери каналів 1, 2 (A/B), Mute, кнопки FX/AUX/CUE (GPx7); внутрішні підтяжки 100k, INTA/INTB дзеркальні → один INT"
- note removed: "MCP23017 #2 (I²C2, 0x21): енкодери каналів 3, 4 (A/B), Mute, кнопки FX/AUX/CUE (GPx7); внутрішні підтяжки 100k, INTA/INTB дзеркальні → один INT"
- note removed: "USB-C (GCT USB4085, з Rev A): аудіо, MIDI, заряд. CC 5,1k — пристрій-споживач; ESD USBLC6"
- note removed: "Канал 1: 3 енкодери EC11 (шари EQ / посили / канал, DM6), фейдер 35 мм (DM8), Mute — тактова кнопка TSF-1266 (DM16)"
- note removed: "Канал 2: 3 енкодери EC11 (шари EQ / посили / канал, DM6), фейдер 35 мм (DM8), Mute — тактова кнопка TSF-1266 (DM16)"
- note removed: "Канал 3: 3 енкодери EC11 (шари EQ / посили / канал, DM6), фейдер 35 мм (DM8), Mute — тактова кнопка TSF-1266 (DM16)"
- note removed: "Канал 4: 3 енкодери EC11 (шари EQ / посили / канал, DM6), фейдер 35 мм (DM8), Mute — тактова кнопка TSF-1266 (DM16)"
- note removed: "Майстер: енкодер EC11 з кнопкою, кнопки FX I, FX II, AUX, CUE, SHIFT (TSF-1266); дисплей GMT147SPI 1,47" 172×320 ST7789P3, SPI, на гребінці (DM18, DM23); виводи — за кресленням продавця"

Commit message: digital-mixer: 4 шари (DM31), пара USB D+/D- наперед, розводка 0 помилок
- плата 4 шари як Rev A: F сигнали / In1 GND / In2 сигнали й живлення / B сигнали; доріжки 0,2 мм
- USB D+/D- прокладено парою 0,2/0,2 мм над In1 (92,5 / 90,9 мм) і зафіксовано до автороутера
- кнопки правої колонки повернуті площадкою GND до пари; конденсатори накачки й вихідні
  470 Ом ЦАП, конденсатори TPA6132A2 - біля виводів; TPA6132A2 розвернута до PHONES
- common: patch_route --ignore, fix_pcb --no-cleanup і переходи в острівці GND, кінці доріжок у
  переходах не вважаються висячими, виправлено падіння на видалених переходах
- DRC: 0 порушень, 0 нез'єднаних, 0 розбіжностей зі схемою; ERC 0

Co-Authored-By: Claude Opus 5.5 <noreply@anthropic.com>
Parts:
- C36, C37, R41, R42: Decouples (none) -> U8
- C47, C48, R43, R44: Decouples (none) -> U9
- C58, C59, R45, R46: Decouples (none) -> U10

Commit message: digital-mixer: Teensy на гребінках з PSRAM (DM35), прошивка 0.2, GPL-3.0 (DM36)
Плата: Teensy 4.1 на гребінках у наскрізні отвори (зазор 2,5 мм під PSRAM),
D-/D+ теж наскрізні, Teensy за 6 мм від переднього краю, бокові джеки з кроком
12,5 мм, лапки EC12SY укорочено; перерозведено - DRC 0 порушень, 0 розривів.
Gerber, BOM і файли NextPCB оновлено.

Прошивка: метри каналів після фейдера (CLIP - лише вхід АЦП), калібрування
фейдерів, SHIFT HOLD/TOGGLE, MASTER = AUX у шарі AUX, кроки гучностей,
виправлено EQ на мінімумі, піктограма батареї, назви FX на екрані; збірка
uac2 (UAC2 8x8, 48 kHz) через tools/setup_uac2.sh.

Ліцензія digital-mixer/ - GPL-3.0-or-later.

Co-Authored-By: Claude Opus 5.5 <noreply@anthropic.com>
Parts:
- U1: footprint pocket-digital:Teensy41_SMD -> pocket-digital:Teensy41_THT
Other:
- note added: "Teensy 4.1 (DM4, DM12, DM35): на гребінках 2 × 24 крізь плату, зазор 2,5 мм під PSRAM; VIN = +4V2; перемичку VIN–VUSB на модулі РОЗРІЗАТИ, VUSB = VBUS з USB-C; USB device D−/D+ — отвори знизу модуля (креслення PJRC) → площадки 66/67 під ними, VUSB — дротик (49)"
- note removed: "Teensy 4.1 (DM4, DM12): VIN = +4V2; перемичку VIN–VUSB на модулі РОЗРІЗАТИ, VUSB = VBUS з USB-C; USB device — площадки D+/D− знизу (66/67, XenGi teensy_library; звірити з PJRC)"

Commit message: digital-mixer: перевірка перед замовленням (07-review): +3V3A у межах LP5907 (DM37), переходи з площадок, дроти USB Teensy, USB-живлення в прошивці
Co-Authored-By: Claude Opus 5.5 <noreply@anthropic.com>
Parts:
- C11: value 10u -> 2.2u
- C18, C30, C41, C52, C63: value 10u -> 1u
Other:
- note added: "LP5907 3,3 V — аналог кодеків (+3V3A): < 6,5 µVrms, 250 mA; навантаження 128 mA (calc/power.py). Ємність на всій шині +3V3A — 0,7…10 µF (datasheet, COUT): 2,2 µF тут + 1 µF біля кожного кодека + 100 nF ≈ 8 µF"
- note removed: "LP5907 3,3 V — аналог кодеків (+3V3A): < 6,5 µVrms, 250 mA; навантаження 128 mA (calc/power.py)"
