File: digital-mixer/hw/main/main.kicad_sch (KiCad schematic)
At the start: 186 parts, among them J1 GCT USB4110-GF-A, J10 MIDI OUT SJ-43514-SMT, J2 LiPo 1S 3000 mAh (з платою за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, J3 IN1 SJ-43514-SMT, J4 IN2 SJ-43514-SMT, J5 IN3 SJ-43514-SMT, J6 IN4 SJ-43514-SMT, J7 MAIN OUT SJ-43514-SMT, J8 AUX OUT SJ-43514-SMT, J9 PHONES SJ-43514-SMT, Q1 AO3401A, SW1 Power 5.8mm DPDT self-lock SMD, SW10 EC12SY ch3.1, SW11 EC12SY ch3.2, SW12 EC12SY ch3.3, SW13 Mute 3 TSF-1266, SW14 EC12SY ch4.1, SW15 EC12SY ch4.2, SW16 EC12SY ch4.3, SW17 Mute 4 TSF-1266, SW18 EC12SY master, SW19 FX1 TSF-1266, SW2 EC12SY ch1.1, SW20 FX2 TSF-1266, SW21 AUX TSF-1266, SW22 SHIFT TSF-1266, SW3 EC12SY ch1.2, SW4 EC12SY ch1.3, SW5 Mute 1 TSF-1266, SW6 EC12SY ch2.1, SW7 EC12SY ch2.2, SW8 EC12SY ch2.3, SW9 Mute 2 TSF-1266, U1 Teensy 4.1, U10 PCM5102A, U11 TPA6132A2, U12 MCP23017-E/SO, U13 MCP23017-E/SO, U14 MCP23017-E/SO, U2 USBLC6-2SC6, U3 TP4056, U4 TPS63802, U5 LP5907MFX-3.3, U6 PCM1865, U7 PCM1865, U8 PCM5102A, U9 PCM5102A

Commit message: digital-mixer: джеки PJ-327A замість SJ-43514 (DM38)
- footprint, 3D-модель і символ за кресленням продавця AliExpress (площадки 5 × 2 × 3, контакти:
  4 кінчик, 3 кільце, 1 / 2 гільза, 5 перемикач — вільний); креслення HOOYA / XKB / SOFNG — для звірки
- розведена плата: 8 джеків замінено латками, передній торець по краю, носик 2 мм назовні; J8 зсунуто
  на 0,4 мм (напрямна біля кнопки AUX); заборонні зони під нові отвори; DRC 0, розривів 0, схема 0, ERC 0
- джеки — ручний монтаж у всіх варіантах NextPCB (PJ-327A інших виробників мають інші лапки)
- кошик AliExpress на 1 плату: ≈ 400 грн замість 959

Co-Authored-By: Claude Opus 5.5 <noreply@anthropic.com>
Parts:
- removed J10: MIDI OUT SJ-43514-SMT, pocket-digital:CUI_SJ-43514-SMT_TRRS_Horizontal, symbol pocket-digital:AudioJack_TRRS_SJ-43514
- removed J3: IN1 SJ-43514-SMT, pocket-digital:CUI_SJ-43514-SMT_TRRS_Horizontal, symbol pocket-digital:AudioJack_TRRS_SJ-43514
- removed J4: IN2 SJ-43514-SMT, pocket-digital:CUI_SJ-43514-SMT_TRRS_Horizontal, symbol pocket-digital:AudioJack_TRRS_SJ-43514
- removed J5: IN3 SJ-43514-SMT, pocket-digital:CUI_SJ-43514-SMT_TRRS_Horizontal, symbol pocket-digital:AudioJack_TRRS_SJ-43514
- removed J6: IN4 SJ-43514-SMT, pocket-digital:CUI_SJ-43514-SMT_TRRS_Horizontal, symbol pocket-digital:AudioJack_TRRS_SJ-43514
- removed J7: MAIN OUT SJ-43514-SMT, pocket-digital:CUI_SJ-43514-SMT_TRRS_Horizontal, symbol pocket-digital:AudioJack_TRRS_SJ-43514
- removed J8: AUX OUT SJ-43514-SMT, pocket-digital:CUI_SJ-43514-SMT_TRRS_Horizontal, symbol pocket-digital:AudioJack_TRRS_SJ-43514
- removed J9: PHONES SJ-43514-SMT, pocket-digital:CUI_SJ-43514-SMT_TRRS_Horizontal, symbol pocket-digital:AudioJack_TRRS_SJ-43514
- added J10: MIDI OUT PJ-327A, pocket-digital:Jack_3.5mm_PJ-327A_SMT_Horizontal, symbol pocket-digital:AudioJack_Stereo_PJ-327A
- added J3: IN1 PJ-327A, pocket-digital:Jack_3.5mm_PJ-327A_SMT_Horizontal, symbol pocket-digital:AudioJack_Stereo_PJ-327A
- added J4: IN2 PJ-327A, pocket-digital:Jack_3.5mm_PJ-327A_SMT_Horizontal, symbol pocket-digital:AudioJack_Stereo_PJ-327A
- added J5: IN3 PJ-327A, pocket-digital:Jack_3.5mm_PJ-327A_SMT_Horizontal, symbol pocket-digital:AudioJack_Stereo_PJ-327A
- added J6: IN4 PJ-327A, pocket-digital:Jack_3.5mm_PJ-327A_SMT_Horizontal, symbol pocket-digital:AudioJack_Stereo_PJ-327A
- added J7: MAIN OUT PJ-327A, pocket-digital:Jack_3.5mm_PJ-327A_SMT_Horizontal, symbol pocket-digital:AudioJack_Stereo_PJ-327A
- added J8: AUX OUT PJ-327A, pocket-digital:Jack_3.5mm_PJ-327A_SMT_Horizontal, symbol pocket-digital:AudioJack_Stereo_PJ-327A
- added J9: PHONES PJ-327A, pocket-digital:Jack_3.5mm_PJ-327A_SMT_Horizontal, symbol pocket-digital:AudioJack_Stereo_PJ-327A
Connections:
- net AUX_L: now also J8.4 (T)
- net AUX_R: now also J8.3 (R)
- net GND: now also J10.1 (S), J10.2 (S2), J3.1 (S), J3.2 (S2), J4.1 (S), J4.2 (S2), J5.1 (S), J5.2 (S2), J6.1 (S), J6.2 (S2), J7.1 (S), J7.2 (S2), J8.1 (S), J8.2 (S2), J9.1 (S), J9.2 (S2)
- net IN1_R: now also J3.3 (R)
- net IN1_T: now also J3.4 (T)
- net IN2_R: now also J4.3 (R)
- net IN2_T: now also J4.4 (T)
- net IN3_R: now also J5.3 (R)
- net IN3_T: now also J5.4 (T)
- net IN4_R: now also J6.3 (R)
- net IN4_T: now also J6.4 (T)
- net MAIN_L: now also J7.4 (T)
- net MAIN_R: now also J7.3 (R)
- net MIDI_SINK: now also J10.4 (T)
- net MIDI_SRC: now also J10.3 (R)
- net PH_L: now also J9.4 (T)
- net PH_R: now also J9.3 (R)
- no-connect marks 63 -> 71

Commit message: digital-mixer: фейдери Alps RS201111J011 замість Bourns PTA2043 (DM39)
Footprint і 3D-модель за кресленням № 1 каталогу Alps (і продавця): 3 виводи Ø1,5,
25 і 3,75 мм. Центр ходу на старому місці; на розведеній платі R12/R13/R48 зсунуто,
38 з'єднань проведено заново. ERC 0, DRC 0 порушень, 0 розривів, 0 розбіжностей.

Co-Authored-By: Claude Opus 5.5 <noreply@anthropic.com>
Parts:
- RV1, RV2, RV3, RV4: value PTA2043 10k B -> RS201111J011 10k B; footprint Potentiometer_THT:Potentiometer_Bourns_PTA2043_Single_Slide -> pocket-digital:Potentiometer_Alps_RS20111_Single_Slide
Other:
- note added: "Канал 1: 3 енкодери EC12SY SMD з кнопкою (шари EQ / посили / канал, DM6, DM26), фейдер 35 мм Alps RS201111J011 (DM8, DM39), Mute — тактова кнопка TSF-1266 (DM16)"
- note added: "Канал 2: 3 енкодери EC12SY SMD з кнопкою (шари EQ / посили / канал, DM6, DM26), фейдер 35 мм Alps RS201111J011 (DM8, DM39), Mute — тактова кнопка TSF-1266 (DM16)"
- note added: "Канал 3: 3 енкодери EC12SY SMD з кнопкою (шари EQ / посили / канал, DM6, DM26), фейдер 35 мм Alps RS201111J011 (DM8, DM39), Mute — тактова кнопка TSF-1266 (DM16)"
- note added: "Канал 4: 3 енкодери EC12SY SMD з кнопкою (шари EQ / посили / канал, DM6, DM26), фейдер 35 мм Alps RS201111J011 (DM8, DM39), Mute — тактова кнопка TSF-1266 (DM16)"
- note removed: "Канал 1: 3 енкодери EC12SY SMD з кнопкою (шари EQ / посили / канал, DM6, DM26), фейдер 35 мм (DM8), Mute — тактова кнопка TSF-1266 (DM16)"
- note removed: "Канал 2: 3 енкодери EC12SY SMD з кнопкою (шари EQ / посили / канал, DM6, DM26), фейдер 35 мм (DM8), Mute — тактова кнопка TSF-1266 (DM16)"
- note removed: "Канал 3: 3 енкодери EC12SY SMD з кнопкою (шари EQ / посили / канал, DM6, DM26), фейдер 35 мм (DM8), Mute — тактова кнопка TSF-1266 (DM16)"
- note removed: "Канал 4: 3 енкодери EC12SY SMD з кнопкою (шари EQ / посили / канал, DM6, DM26), фейдер 35 мм (DM8), Mute — тактова кнопка TSF-1266 (DM16)"
